File: driven-amplifier-board/driven-amplifier-board.kicad_pcb (KiCad board)
At the start: 2 copper layers, 58 x 35.5 mm, 5 parts, among them J1 Conn_Coaxial, U1 Teyleten-Differential-Amplifi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

Commit message: Saving some old modifications.
Connections:
- BatteryPower1 pad 2: Net-(BatteryPower1-Pad2) -> GND
- J1 pad 2: Net-(J1-Pad2) -> GND
- U1 pad 3: Net-(BatteryPower1-Pad2) -> GND
- U1 pad 6: Net-(J1-Pad2) -> GND
Routing:
- net Net-(BatteryPower1-Pad2): track 15.6 -> 0.00 mm
- net Net-(J1-Pad2): track 10.3 -> 0.00 mm
Changed lines of the file:
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@@
     (thickness 1.6)
     (drawings 4)
-    (tracks 12)
+    (tracks 9)
     (zones 0)
     (modules 5)
-    (nets 8)
+    (nets 7)
   )
   (page A4)
@@
       (usegerberattributes true)
       (usegerberadvancedattributes true)
-      (creategerberjobfile true)
+      (creategerberjobfile false)
       (excludeedgelayer true)
       (linewidth 0.100000)
@@
   )
   (net 0 "")
-  (net 1 "Net-(BatteryPower1-Pad2)")
-  (net 2 "Net-(BatteryPower1-Pad1)")
-  (net 3 "Net-(J1-Pad2)")
-  (net 4 "Net-(J1-Pad1)")
-  (net 5 GND)
-  (net 6 "Net-(S+1-Pad1)")
-  (net 7 "Net-(S-1-Pad1)")
+  (net 1 "Net-(BatteryPower1-Pad1)")
+  (net 2 "Net-(J1-Pad2)")
+  (net 3 "Net-(J1-Pad1)")
+  (net 4 GND)
+  (net 5 "Net-(S+1-Pad1)")
+  (net 6 "Net-(S-1-Pad1)")
   (net_class Default "This is the default net class."
     (clearance 0.75)
@@
     (add_net GND)
     (add_net "Net-(BatteryPower1-Pad1)")
-    (add_net "Net-(BatteryPower1-Pad2)")
     (add_net "Net-(J1-Pad1)")
     (add_net "Net-(J1-Pad2)")
@@
     (fp_line (start -9.7 37.25) (end -9.7 5) (layer F.SilkS) (width 0.12))
     (pad 6 thru_hole circle (at -0.003333 34.725) (size 1.524 1.524) (drill 0.762) (layers *.Cu *.Mask)
-      (net 3 "Net-(J1-Pad2)"))
+      (net 4 GND))
     (pad 5 thru_hole circle (at 2.523333 34.725 90) (size 1.524 1.524) (drill 0.762) (layers *.Cu *.Mask)
-      (net 4 "Net-(J1-Pad1)"))
+      (net 3 "Net-(J1-Pad1)"))
     (pad 4 thru_hole circle (at -2.53 6.6 180) (size 1.524 1.524) (drill 0.762) (layers *.Cu *.Mask)
-      (net 2 "Net-(BatteryPower1-Pad1)"))
+      (net 1 "Net-(BatteryPower1-Pad1)"))
     (pad 3 thru_hole circle (at -0.003333 6.6) (size 1.524 1.524) (drill 0.762) (layers *.Cu *.Mask)
-      (net 1 "Net-(BatteryPower1-Pad2)"))
+      (net 4 GND))
     (pad 2 thru_hole circle (at 2.523333 6.6 90) (size 1.524 1.524) (drill 0.762) (layers *.Cu *.Mask)
-      (net 7 "Net-(S-1-Pad1)"))
+      (net 6 "Net-(S-1-Pad1)"))
     (pad 1 thru_hole circle (at 5.05 6.6 90) (size 1.524 1.524) (drill 0.762) (layers *.Cu *.Mask)
-      (net 6 "Net-(S+1-Pad1)"))
+      (net 5 "Net-(S+1-Pad1)"))
   )
   (module custom-footprints:amazon-sma-connector (layer F.Cu)
@@
     (fp_poly (pts (xy 0.5 8) (xy -8 8) (xy -8 3) (xy 0.5 3)) (layer F.SilkS) (width 0.1))
     (pad 2 connect rect (at 3 8) (size 5 1) (layers F.Cu F.Mask)
-      (net 5 GND))
+      (net 4 GND))
     (pad 1 connect rect (at 3 5.5) (size 5 1) (layers F.Cu F.Mask)
-      (net 7 "Net-(S-1-Pad1)"))
+      (net 6 "Net-(S-1-Pad1)"))
     (pad 2 connect rect (at 3 3) (size 5 1) (layers F.Cu F.Mask)
-      (net 5 GND))
+      (net 4 GND))
   )
   (module custom-footprints:amazon-sma-connector (layer F.Cu)
@@
     (fp_poly (pts (xy 0.5 8) (xy -8 8) (xy -8 3) (xy 0.5 3)) (layer F.SilkS) (width 0.1))
     (pad 2 connect rect (at 3 8) (size 5 1) (layers F.Cu F.Mask)
-      (net 5 GND))
+      (net 4 GND))
     (pad 1 connect rect (at 3 5.5) (size 5 1) (layers F.Cu F.Mask)
-      (net 6 "Net-(S+1-Pad1)"))
+      (net 5 "Net-(S+1-Pad1)"))
     (pad 2 connect rect (at 3 3) (size 5 1) (layers F.Cu F.Mask)
-      (net 5 GND))
+      (net 4 GND))
   )
   (module custom-footprints:amazon-sma-connector (layer F.Cu)
@@
     (fp_poly (pts (xy 0.5 8) (xy -8 8) (xy -8 3) (xy 0.5 3)) (layer F.SilkS) (width 0.1))
     (pad 2 connect rect (at 3 8 180) (size 5 1) (layers F.Cu F.Mask)
-      (net 3 "Net-(J1-Pad2)"))
+      (net 2 "Net-(J1-Pad2)"))
     (pad 1 connect rect (at 3 5.5 180) (size 5 1) (layers F.Cu F.Mask)
-      (net 4 "Net-(J1-Pad1)"))
+      (net 3 "Net-(J1-Pad1)"))
     (pad 2 connect rect (at 3 3 180) (size 5 1) (layers F.Cu F.Mask)
-      (net 3 "Net-(J1-Pad2)"))
+      (net 4 GND))
   )
   (module TerminalBlock:TerminalBlock_bornier-2_P5.08mm (layer F.Cu)
@@
     (fp_line (start 7.79 4) (end -2.71 4) (layer F.CrtYd) (width 0.05))
     (pad 2 thru_hole circle (at 5.08 0 90) (size 3 3) (drill 1) (layers *.Cu *.Mask)
-      (net 1 "Net-(BatteryPower1-Pad2)"))
+      (net 4 GND))
     (pad 1 thru_hole rect (at 0 0 90) (size 3 3) (drill 1) (layers *.Cu *.Mask)
-      (net 2 "Net-(BatteryPower1-Pad1)"))
+      (net 1 "Net-(BatteryPower1-Pad1)"))
     (model ${KISYS3DMOD}/TerminalBlock.3dshapes/TerminalBlock_bornier-2_P5.08mm.wrl
       (offset (xyz 2.539999961853027 0 0))
@@
   (gr_line (start 23 16.5) (end 81 16.5) (layer Edge.Cuts) (width 0.05))
   (gr_line (start 23 52) (end 23 16.5) (layer Edge.Cuts) (width 0.05))
-  (segment (start 31.183333 43.92) (end 39.6 35.503333) (width 1) (layer F.Cu) (net 1))
-  (segment (start 27.5 43.92) (end 31.183333 43.92) (width 1) (layer F.Cu) (net 1))
-  (segment (start 28.63 49) (end 39.6 38.03) (width 1) (layer F.Cu) (net 2))
-  (segment (start 27.5 49) (end 28.63 49) (width 0.5) (layer F.Cu) (net 2))
-  (segment (start 77.996667 35.503333) (end 78 35.5) (width 0.5) (layer F.Cu) (net 3))
-  (segment (start 67.725 35.503333) (end 77.996667 35.503333) (width 1) (layer F.Cu) (net 3))
-  (segment (start 77.976667 32.976667) (end 78 33) (width 0.5) (layer F.Cu) (net 4))
-  (segment (start 67.725 32.976667) (end 77.976667 32.976667) (width 1) (layer F.Cu) (net 4))
-  (segment (start 29.65 20.5) (end 39.6 30.45) (width 1) (layer F.Cu) (net 6))
-  (segment (start 25.5 20.5) (end 29.65 20.5) (width 1) (layer F.Cu) (net 6))
-  (segment (start 39.576667 33) (end 39.6 32.976667) (width 0.5) (layer F.Cu) (net 7))
-  (segment (start 25.5 33) (end 39.576667 33) (width 1) (layer F.Cu) (net 7))
-  (zone (net 5) (net_name GND) (layer F.Cu) (hatch edge 0.508)
+  (segment (start 28.63 49) (end 39.6 38.03) (width 1) (layer F.Cu) (net 1))
+  (segment (start 27.5 49) (end 28.63 49) (width 0.5) (layer F.Cu) (net 1))
+  (segment (start 77.996667 35.503333) (end 78 35.5) (width 0.5) (layer F.Cu) (net 4))
+  (segment (start 77.976667 32.976667) (end 78 33) (width 0.5) (layer F.Cu) (net 3))
+  (segment (start 67.725 32.976667) (end 77.976667 32.976667) (width 1) (layer F.Cu) (net 3))
+  (segment (start 29.65 20.5) (end 39.6 30.45) (width 1) (layer F.Cu) (net 5))
+  (segment (start 25.5 20.5) (end 29.65 20.5) (width 1) (layer F.Cu) (net 5))
+  (segment (start 39.576667 33) (end 39.6 32.976667) (width 0.5) (layer F.Cu) (net 6))
+  (segment (start 25.5 33) (end 39.576667 33) (width 1) (layer F.Cu) (net 6))
+  (zone (net 4) (net_name GND) (layer F.Cu) (hatch edge 0.508)
     (connect_pads (clearance 0.508))
     (min_thickness 0.254)
